File: Curing Oven HW/Electrical/Curing_Oven_PCBs/UV_Curing-PCB.sch (EAGLE design)
At the start: 18 parts, among them J1 12V_SUP, J2 PINHEADER-5POS-2.54MM, J3 PINHEADER-7POS-2.54MM, J4 UV_SUP, J5 UV_FN, J6 MOTOR, J7 5V_SUP, J8 SPKR, K1 25V, Q1 55V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

Commit message: Updated PCB for fab manufacturing
Parts:
- added D3, D4, D5: 400V, Up3D Active Components:DIODE-DO-41-TH
- added M1, M2, M3, M4: MOUNTING_HOLE, Up3D Misc:MOUNTING_HOLE
- added R4: 1K, Up3D Resistors:MFR-25FBF52-1K
- J1: value 12V_SUP -> PINHEADER-2POS-2.54MM
- J2: value PINHEADER-5POS-2.54MM -> PINHEADER-2POS-2.54MM; device Up3D Misc:PINHEADER-5POS-2.54MM -> Up3D Misc:PINHEADER-2POS-2.54MM
- J3: value PINHEADER-7POS-2.54MM -> PINHEADER-5POS-2.54MM; device Up3D Misc:PINHEADER-7POS-2.54MM -> Up3D Misc:PINHEADER-5POS-2.54MM
- J4: value UV_SUP -> PINHEADER-7POS-2.54MM; device Up3D Misc:PINHEADER-2POS-2.54MM -> Up3D Misc:PINHEADER-7POS-2.54MM
- J5: value UV_FN -> PINHEADER-2POS-2.54MM
- J6: value MOTOR -> PINHEADER-2POS-2.54MM
- J7: value 5V_SUP -> PINHEADER-2POS-2.54MM
- J8: value SPKR -> PINHEADER-2POS-2.54MM
- Q3: value 30V 100mA -> 55V; device Up3D Active Components:BJT-NPN -> Up3D Active Components:MOSFET-NCH-TO-220AB-TH
- R1: value 220E -> 1K
- R3: value 10K -> 8E
Connections:
- net MOTOR_SW renamed MOT_SW
- removed net DI_KEY: J2.4, U1.D2
- removed net DI_S1: J2.2, U1.A0
- removed net DI_S2: J2.3, U1.A1
- removed net SPEAKER_SW: R1.2, U1.D3
- removed net UV_SW: Q2.G, U1.D5
- new net ENC_KEY: J3.2, U1.D2
- new net ENC_S1: J3.4, U1.A1
- new net ENC_S2: J3.3, U1.A0
- new net LAMP_EN: R1.1, U1.D5
- new net N$6: D5.C, J8.1, R3.1
- new net N$9: Q3.G, R4.2
- new net SPK_SW: R4.1, U1.D3
- net +12V: now also D3.C, D4.C, J1.2, J7.1, K1.COIL_1, K1.COM; no longer D1.C, D2.C, J1.02, J5.01, J6.01, K1.COIL_2, K1.NO
- net +5V: now also J2.2, J3.1, J4.6, R3.2; no longer J2.5, J3.6, J7.02, J8.01
- net GND: now also D1.A, D2.A, J1.1, J3.5, J4.7, J5.2, J6.2, Q3.S; no longer J1.01, J3.7, J4.02, J7.01, Q3.E, R3.1
- net N$1: now also Q1.G, R1.2; no longer D1.A, J6.02, Q1.D
- net N$2: now also D1.C, D2.C, J5.1, J6.1, K1.NO; no longer J4.01, K1.COM
- net N$3: now also D3.A, K1.COIL_2, Q1.D; no longer Q1.G, R2.2, R3.2
- net N$4: now also Q2.G, R2.2; no longer D2.A, J5.02, K1.COIL_1, Q2.D
- net N$5: now also D4.A, J7.2, Q2.D; no longer J8.02, Q3.C
- net N$7: now also D5.A, J8.2, Q3.D; no longer Q3.B, R1.1
- net OLED_CLK: now also J4.5; no longer J3.5
- net OLED_CS: now also J4.1; no longer J3.1
- net OLED_DC: now also J4.2; no longer J3.2
- net OLED_MOSI: now also J4.4; no longer J3.4
- net OLED_RST: now also J4.3; no longer J3.3
Other:
- note added: "12V Input Header"
- note added: "5 x RC time constant = 7.43us Max switching freq = 68kHz For higher freq use smaller resistor"
- note added: "5V Input Header"
- note added: "Arduino Nano"
- note added: "Encoder Knob Header"
- note added: "Motor"
- note added: "Mounting Holes to be placed in a 57x86mm square"
- note added: "OLED Header"
- note added: "Power Input"
- note added: "R3 is the volume setting resistor. Lower values will result in louder volumes"
- note added: "Speaker"
- note added: "UI Headers"
- note added: "UV Lamp"
- note added: "UV Lamp Fan"
- note added: "UV Lamp Supply 36V Boost Converter"
- moved on the sheet: Q1, Q2, R1, R2, R3, U1
